File: hw/evopower/mjpower_ss.kicad_sch (KiCad schematic)
At the start: 28 parts, among them J1 Conn_01x02_Pin, J2 Conn_01x04_Pin, P1 Conn_01x02_Pin, P7 XT60, Q1 PSMN3R7-100BSEJ, Q2 PSMN3R7-100BSEJ, Q3 PSMN3R7-100BSEJ, SW1 SW_SPDT, U1 TPS2490DGSR, U2 ZXTR2005Z, U3 INA226AIDGSR

Commit message: I really should get better about this
Parts:
- removed Q3: PSMN3R7-100BSEJ, footprints:TRANS_PSMN3R7-100BSEJ, symbol PSMN3R7-100BSEJ:PSMN3R7-100BSEJ
- added C5: C_Small, symbol Device:C_Small
- added J3: Conn_01x01_Pin, symbol Connector:Conn_01x01_Pin
- R3: MPN WSLF2512L5000FEA -> WSLF25121L000FEA
Connections:
- net GND: now also U3.1 (A1), U3.2 (A0), C5.2
- net SENSE: now also U3.8 (VBUS)
- net at U3.6 (VS): now also C5.1, J3.1 (Pin_1)
